Commit message: add launch rviz

File: src/puma560_description/urdf/puma560_robot.urdf.xacro (robot description, xacro)
@@ -3,5 +3,5 @@
     <xacro:property name="mesh_dir" value="package://puma560_description/meshes"/>
     <xacro:macro name="puma560_link_geometry" params="link_num">
-        <mesh filename="${mesh_dir}/puma_link${link_num}.stl" scale="${0.001*25.4} ${0.001*25.4} ${25.4*0.001}"/>
+        <mesh filename="${mesh_dir}/puma_link${link_num}.stl" scale="${0.1*25.4} ${0.1*25.4} ${0.1*25.4}"/>
     </xacro:macro>
     <material name="blue">
@@ -27,10 +27,4 @@
     <xacro:property name="a_5" value="0"/>
     <xacro:property name="a_6" value="0"/>
-    <link name="world"/>
-    <joint name="world_to_link1" type="fixed">
-        <parent link="world"/>
-        <child link="link1"/>
-        <origin xyz="0 0 0" rpy="0 0 0"/>
-    </joint>
     <xacro:macro name="link" params="num color vxyz vrpy cxyz crpy ixyz irpy mass ixx ixy ixz iyy iyz izz">
       <link name="link${num}">
@@ -65,4 +59,5 @@
         </joint>
     </xacro:macro>
+    <link name="world"/>
     <xacro:link num="1" color="green"
                 vxyz="0 0 0" vrpy="0 0 ${M_PI/2}"

Commit message: add simulation

File: src/puma560_description/urdf/puma560_robot.urdf.xacro (robot description, xacro)
@@ -157,6 +157,7 @@
         <parent link="world"/>
         <child link="link1"/>
-    </joint>
-    <joint name="join1" type="revolute">
+        <origin xyz="0 0 0" rpy="0 0 0"/>
+    </joint>
+    <joint name="joint1" type="revolute">
         <parent link="link1"/>
         <child link="link2"/>
@@ -166,5 +167,5 @@
         <dynamics damping="1.0" friction="0.1"/>
     </joint>
-    <joint name="join2" type="revolute">
+    <joint name="joint2" type="revolute">
         <parent link="link2"/>
         <child link="link3"/>
@@ -174,5 +175,5 @@
         <dynamics damping="1.0" friction="0.1"/>
     </joint>
-    <joint name="join3" type="revolute">
+    <joint name="joint3" type="revolute">
         <parent link="link3"/>
         <child link="link4"/>
@@ -182,5 +183,5 @@
         <dynamics damping="1.0" friction="0.1"/>
     </joint>
-    <joint name="join4" type="revolute">
+    <joint name="joint4" type="revolute">
         <parent link="link4"/>
         <child link="link5"/>
@@ -190,5 +191,5 @@
         <dynamics damping="1.0" friction="0.1"/>
     </joint>
-    <joint name="join5" type="revolute">
+    <joint name="joint5" type="revolute">
         <parent link="link5"/>
         <child link="link6"/>
@@ -198,5 +199,5 @@
         <dynamics damping="1.0" friction="0.1"/>
     </joint>
-    <joint name="join6" type="revolute">
+    <joint name="joint6" type="revolute">
         <parent link="link6"/>
         <child link="link7"/>
@@ -206,3 +207,43 @@
         <dynamics damping="1.0" friction="0.1"/>
     </joint>
+    <ros2_control name="GazeboSimSystem" type="system">
+        <hardware>
+            <plugin>gz_ros2_control/GazeboSimSystem</plugin>
+        </hardware>
+        <joint name="joint1">
+            <command_interface name="position"/>
+            <state_interface name="position"/>
+            <state_interface name="velocity"/>
+        </joint>
+        <joint name="joint2">
+            <command_interface name="position"/>
+            <state_interface name="position"/>
+            <state_interface name="velocity"/>
+        </joint>
+        <joint name="joint3">
+            <command_interface name="position"/>
+            <state_interface name="position"/>
+            <state_interface name="velocity"/>
+        </joint>
+        <joint name="joint4">
+            <command_interface name="position"/>
+            <state_interface name="position"/>
+            <state_interface name="velocity"/>
+        </joint>
+        <joint name="joint5">
+            <command_interface name="position"/>
+            <state_interface name="position"/>
+            <state_interface name="velocity"/>
+        </joint>
+        <joint name="joint6">
+            <command_interface name="position"/>
+            <state_interface name="position"/>
+            <state_interface name="velocity"/>
+        </joint>
+    </ros2_control>
+    <gazebo>
+        <plugin filename="gz_ros2_control-system" name="gz_ros2_control::GazeboSimROS2ControlPlugin">
+            <parameters>$(find puma560_description)/config/controllers.yaml</parameters>
+        </plugin>
+    </gazebo>
 </robot>

Commit message: angle correction

File: src/puma560_description/urdf/puma560_robot.urdf.xacro (robot description, xacro)
@@ -172,5 +172,5 @@
         <origin xyz="0 0 0" rpy="0 0 0"/>
         <axis xyz="0 0 1"/>
-        <limit effort="1000.0" lower="-1.570796325" upper="1.570796325" velocity="2.0"/>
+        <limit effort="1000.0" lower="-0.8552113325" upper="3.9968039825" velocity="2.0"/>
         <dynamics damping="1.0" friction="0.1"/>
     </joint>
@@ -180,5 +180,5 @@
         <origin xyz="0.4318 -0.0203 0.1501" rpy="0 0 -1.570796325"/>
         <axis xyz="0 0 1"/>
-        <limit effort="1000.0" lower="-1.570796325" upper="1.570796325" velocity="2.0"/>
+        <limit effort="1000.0" lower="-0.8552113325" upper="3.9968039825" velocity="2.0"/>
         <dynamics damping="1.0" friction="0.1"/>
     </joint>
@@ -188,5 +188,5 @@
         <origin xyz="0 0 0" rpy="1.570796325 0 1.570796325"/>
         <axis xyz="0 0 1"/>
-        <limit effort="1000.0" lower="-1.570796325" upper="1.570796325" velocity="2.0"/>
+        <limit effort="1000.0" lower="-3.316125575" upper="2.1816615625" velocity="2.0"/>
         <dynamics damping="1.0" friction="0.1"/>
     </joint>
@@ -196,5 +196,5 @@
         <origin xyz="0 0 0.4331" rpy="1.570796325 0 0"/>
         <axis xyz="0 0 1"/>
-        <limit effort="1000.0" lower="-1.570796325" upper="1.570796325" velocity="2.0"/>
+        <limit effort="1000.0" lower="-1.74532925" upper="1.74532925" velocity="2.0"/>
         <dynamics damping="1.0" friction="0.1"/>
     </joint>
@@ -204,5 +204,5 @@
         <origin xyz="0 0.0558 0" rpy="-1.570796325 0 0"/>
         <axis xyz="0 0 1"/>
-        <limit effort="1000.0" lower="-1.570796325" upper="1.570796325" velocity="2.0"/>
+        <limit effort="1000.0" lower="-3.14159265" upper="3.14159265" velocity="2.0"/>
         <dynamics damping="1.0" friction="0.1"/>
     </joint>

Commit message: .

File: src/puma560_description/urdf/puma560_robot.urdf.xacro (robot description, xacro)
@@ -172,5 +172,5 @@
         <origin xyz="0 0 0" rpy="0 0 0"/>
         <axis xyz="0 0 1"/>
-        <limit effort="1000.0" lower="-0.8552113325" upper="3.9968039825" velocity="2.0"/>
+        <limit effort="1000.0" lower="-0.85521133" upper="3.99680399" velocity="2.0"/>
         <dynamics damping="1.0" friction="0.1"/>
     </joint>
@@ -180,5 +180,5 @@
         <origin xyz="0.4318 -0.0203 0.1501" rpy="0 0 -1.570796325"/>
         <axis xyz="0 0 1"/>
-        <limit effort="1000.0" lower="-0.8552113325" upper="3.9968039825" velocity="2.0"/>
+        <limit effort="1000.0" lower="-0.85521133" upper="3.99680399" velocity="2.0"/>
         <dynamics damping="1.0" friction="0.1"/>
     </joint>
@@ -188,5 +188,5 @@
         <origin xyz="0 0 0" rpy="1.570796325 0 1.570796325"/>
         <axis xyz="0 0 1"/>
-        <limit effort="1000.0" lower="-3.316125575" upper="2.1816615625" velocity="2.0"/>
+        <limit effort="1000.0" lower="-3.31612558" upper="2.18166157" velocity="2.0"/>
         <dynamics damping="1.0" friction="0.1"/>
     </joint>

Commit message: add connection to robot

File: src/puma560_description/urdf/puma560_robot.urdf.xacro (robot description, xacro)
@@ -1,4 +1,5 @@
 <?xml version="1.0"?>
 <robot name="Puma560" xmlns:xacro="http://www.ros.org/wiki/xacro">
+    <xacro:arg name="use_sim_time" default="true"/>
     <xacro:macro name="robot_mesh" params="name">
         <mesh filename="package://puma560_description/meshes/${name}" scale="${0.001*25.4} ${0.001*25.4} ${0.001*25.4}"/>
@@ -172,5 +173,5 @@
         <origin xyz="0 0 0" rpy="0 0 0"/>
         <axis xyz="0 0 1"/>
-        <limit effort="1000.0" lower="-0.8552113325" upper="3.9968039825" velocity="2.0"/>
+        <limit effort="1000.0" lower="-0.85521133" upper="3.99680399" velocity="2.0"/>
         <dynamics damping="1.0" friction="0.1"/>
     </joint>
@@ -180,5 +181,5 @@
         <origin xyz="0.4318 -0.0203 0.1501" rpy="0 0 -1.570796325"/>
         <axis xyz="0 0 1"/>
-        <limit effort="1000.0" lower="-0.8552113325" upper="3.9968039825" velocity="2.0"/>
+        <limit effort="1000.0" lower="-0.85521133" upper="3.99680399" velocity="2.0"/>
         <dynamics damping="1.0" friction="0.1"/>
     </joint>
@@ -188,5 +189,5 @@
         <origin xyz="0 0 0" rpy="1.570796325 0 1.570796325"/>
         <axis xyz="0 0 1"/>
-        <limit effort="1000.0" lower="-3.316125575" upper="2.1816615625" velocity="2.0"/>
+        <limit effort="1000.0" lower="-3.31612558" upper="2.18166157" velocity="2.0"/>
         <dynamics damping="1.0" friction="0.1"/>
     </joint>
@@ -207,7 +208,12 @@
         <dynamics damping="1.0" friction="0.1"/>
     </joint>
-    <ros2_control name="GazeboSimSystem" type="system">
+    <ros2_control name="simulation_system" type="system">
         <hardware>
-            <plugin>gz_ros2_control/GazeboSimSystem</plugin>
+            <xacro:if value="$(arg use_sim_time)">
+                <plugin>gz_ros2_control/GazeboSimSystem</plugin>
+            </xacro:if>
+            <xacro:unless value="$(arg use_sim_time)">
+                <plugin>puma560_description/RobotHardwareInterface</plugin>
+            </xacro:unless>
         </hardware>
         <joint name="joint1">
@@ -242,8 +248,10 @@
         </joint>
     </ros2_control>
-    <gazebo>
-        <plugin filename="gz_ros2_control-system" name="gz_ros2_control::GazeboSimROS2ControlPlugin">
-            <parameters>$(find puma560_description)/config/controllers.yaml</parameters>
-        </plugin>
-    </gazebo>
+    <xacro:if value="$(arg use_sim_time)">
+        <gazebo>
+            <plugin filename="gz_ros2_control-system" name="gz_ros2_control::GazeboSimROS2ControlPlugin">
+                <parameters>$(find puma560_description)/config/controllers.yaml</parameters>
+            </plugin>
+        </gazebo>
+    </xacro:if>
 </robot>
